Commit message: 最终版：夹爪 JTC 直驱 + 前万向轮防前倾 + 抓取自检/TF 间隙判据 + 官方比赛世界
- 夹爪弃 mimic → gripper_controller 换 JTC 直驱两指（gap 60.04mm）；
  限位上下各留 2mm（0.002/0.038）避免 Fortress 越限死锁
- 抓取判据改 TF 实测两指间隙（弃 2×joint1，两指可不对称）；空合→微挪→
  重拍重识别→重抓循环（上限 2）
- 前万向轮 caster_front + gazebo 低摩擦块（mu=0.1），修伸臂时底盘前倾
  11.7°→0.3°（抓取点 0.196m 偏移根因）
- grasp_phase 抓取点自检 _target_suspect，防照偏掉的点下爪
- 视觉置信门/复核调整；insid3_review/vision_pipeline/patrol_task 配套
- 新增官方比赛世界 official-ros2.world，launch 切换到它

File: franka_description/end_effectors/common/franka_hand.xacro (robot description, xacro)
@@ -126,5 +126,16 @@
       <axis xyz="0 1 0" />
       <limit effort="100" lower="0.0" upper="0.04" velocity="0.2" />
-      <mimic joint="${ee_prefix}finger_joint1" />
+      <!-- ★ 2026-09-18 删掉 <mimic joint="...finger_joint1"/>（原来是硬编码到这里的第一关节）。
+           夹爪两指在本工程里必须各自独立受控，而这一行 <mimic> 有三个消费者都会读它 ✗：
+             · MoveIt：把 joint2 当成 passive/mimic 关节 → **从 hand 组的 active joints 里剔除**
+               （`getActiveJointModelNames()` 只剩 fr3_finger_joint1）→ 规划出来的轨迹只有
+               1 个关节名 → JointTrajectoryController 直接拒收
+               （实跑报错：`Joints on incoming trajectory don't match the controller joints.`，
+                MoveIt 侧表现为 `Goal request rejected` / error_code=-4）。★ 主因
+             · Gazebo：URDF→SDF 只输出 SDF 1.7，而 <mimic> 是 1.9 的元素 → 静默丢弃，
+               本来就没生效（gz-sim/DART 也无 mimic 实现）
+             · robot_state_publisher：只在 joint_states 缺该关节时才用 mimic 兜底；
+               现在 /joint_states 里两指都在 → 不影响
+           删掉后 hand 组的 active joints = {joint1, joint2}，两指由同一个 JTC 驱动。 -->
       <dynamics damping="0.3" />
     </joint>

File: turtlebot3_manipulation_gazebo/gazebo/turtlebot3_waffle_pi.gazebo.xacro (robot description, xacro)
@@ -42,4 +42,16 @@
   </gazebo>
   <gazebo reference="${prefix}caster_back_left_link">
+    <mu1>0.1</mu1>
+    <mu2>0.1</mu2>
+    <kp>1000000.0</kp>
+    <kd>100.0</kd>
+    <minDepth>0.001</minDepth>
+    <maxVel>1.0</maxVel>
+    <material>Gazebo/FlatBlack</material>
+  </gazebo>
+  <!-- ★ 2026-09-18 前万向轮的低摩擦块（照抄上面两个后万向轮）。
+       缺这块的话前轮会用 Gazebo 默认摩擦（≈1.0）→ 变成一块高摩擦刹车垫，
+       转向时跟车较劲，还不解决前倾。mu1/mu2=0.1 才是万向轮该有的行为。 -->
+  <gazebo reference="${prefix}caster_front_link">
     <mu1>0.1</mu1>
     <mu2>0.1</mu2>

File: turtlebot3_manipulation_gazebo/ros2_control/turtlebot3_manipulation_system.ros2_control.xacro (robot description, xacro)
@@ -177,12 +177,65 @@
         </state_interface>
       </joint>
-      <!-- FR3 finger (only joint1; joint2 is URDF mimic handled by Gazebo physics) -->
+      <!-- ══════════ FR3 夹爪（两指，各自独立受控）══════════
+           ★ 2026-09-18 起**彻底不用 mimic**，两个手指各自是一个普通受控关节，
+             由同一个 JointTrajectoryController（gripper_controller）驱动。
+           ■ 为什么不用 URDF 的 <mimic>：
+             URDF→SDF 只输出 SDF 1.7，而 <mimic> 是 1.9 的元素 → **静默丢弃**
+             （`gz sdf -p` 零报错、joint2 照旧存在但 mimic 没了），gz-sim/DART 也无实现。
+             后果（09-17 实测）：joint2 成完全自由被动关节，只有 joint1 走全程，
+             两指不对称、夹持中心横移最多 20mm（容差只有 ±6.5mm）。
+           ■ 为什么连 gz_ros2_control 的 mimic 也不用（09-18 实测，这是关键）：
+             在 ros2_control 层挂 `_mimic`+`mimic`+`multiplier` 确实能让两指在
+             **自由空间**同步（日志 "Joint 'fr3_finger_joint2'is mimicking joint
+             'fr3_finger_joint1' with multiplier: 1"，80mm→0mm 约 0.75s），
+             但**一接触实物就失效**——实测 60mm 方块：
+               j1 被方块挡住停在 0.030，j2 明明还有 ~10mm 完全无障碍的行程，
+               却冻在 0.040 一步不走 → gap 70mm = 只碰到一侧，根本没夹住。
+             给它加一个控制器去"认领"命令接口也没用：mimic 关节的命令接口在
+             resource_manager 里被改名成 `<原名>_mimic`（/joint_states 里可看到
+             fr3_finger_joint2_mimic、而且 fr3_finger_joint2 整个消失），
+             且硬件 mimic 在 `write()` 里最后执行、会覆盖控制器的命令。
+             （controller_manager 每周期顺序：read() → 控制器 update() → write() 硬件）
+           ■ 现在的做法：两指都交给 gripper_controller（JTC）直接驱动，
+             MTC 的 MoveTo("open"/"close") 经 moveit_controllers.yaml 下发两指轨迹，
+             各指独立伺服、各自停在物体两侧。同一个 60mm 方块实测：
+               j1=0.03001 j2=0.03003 gap=60.04mm，JTC 返回 SUCCEEDED ✓
+             SRDF 的 hand group 里必须同时包含 fr3_finger_joint1/2，抓取代码
+             `for (jname : jmg->getActiveJointModelNames()) close_goal[jname] = ...`
+             才会自动给两指设同一目标。
+           ■ 限位上下都留 2mm 裕量（command min/max = 0.002/0.038，而非 URDF 的 0/0.04）：
+             gz-sim Fortress 的已知 bug：prismatic 关节越过 URDF 限位后**永久卡死**，
+             任何命令都不再响应（gz_ros2_control #192/#165，Harmonic 才修）。
+             09-18 实测，上下限各踩中一次：
+               · 上限：出生后立即命令到 0.04 → j2 死锁在 0.04000，连发 0.0 都纹丝不动；
+                 而抓取流程第一步恰恰就是 "open hand"（SRDF 的 open 状态原为 0.04）。
+               · 下限：连续开合，合到 0.0 后发 0.038 → j1 死锁在 0.00000、只剩 j2 能走
+                 （error_code -5）。而 pick_and_place.cpp 在物体识别失败（span<=0）时会
+                 回退到 SRDF 的 "close" 状态，原来正是 0.0 —— 一条真实的死锁路径。
+             两次都只能重启仿真才能恢复，所以命令范围收成 [0.002, 0.038]
+             （开口 4~76mm；最薄的比赛目标糖盒 38mm 对应关节 0.0145，远在范围内）。
+             run3 里 j1 停在 0.04016（越限 0.16mm）后死锁，也是同一个 bug。
+             宁可少开/少合 2mm，也不能让开合爪动作把夹爪锁死。
+             SRDF 的 open/close 状态、joint_limits.yaml 的 max/min_position
+             都已同步成 0.038/0.002，改一处要三处一起改。 -->
       <joint name="fr3_finger_joint1">
         <command_interface name="position">
-          <param name="min">0.0</param>
-          <param name="max">0.04</param>
-        </command_interface>
-        <state_interface name="position">
-          <param name="initial_value">0.04</param>
+          <param name="min">0.002</param>
+          <param name="max">0.038</param>
+        </command_interface>
+        <state_interface name="position">
+          <param name="initial_value">0.038</param>
+        </state_interface>
+        <state_interface name="velocity">
+          <param name="initial_value">0.0</param>
+        </state_interface>
+      </joint>
+      <joint name="fr3_finger_joint2">
+        <command_interface name="position">
+          <param name="min">0.002</param>
+          <param name="max">0.038</param>
+        </command_interface>
+        <state_interface name="position">
+          <param name="initial_value">0.038</param>
         </state_interface>
         <state_interface name="velocity">

File: turtlebot3_manipulation_gazebo/urdf/turtlebot3_waffle_pi.urdf.xacro (robot description, xacro)
@@ -134,4 +134,33 @@
     </inertial>
   </link>
+  <!-- ★ 2026-09-18 前万向轮：把支撑多边形前边界从 x=0 推到 x=+0.18。
+       原来两个万向轮都在后方（x=-0.177），前方无支撑点，而 FR3 臂 19.6 kg、
+       质心高 0.87 m（底盘才 1.55 kg）→ 向前伸臂时整车绕驱动轮前倾。
+       实测：臂收回 pitch=-0.15°，伸到抓取位 pitch=+11.55°（Δ=11.7°）。
+       后果：base_footprint 随底盘一起转，而视觉/creep 是在臂收回（pitch≈0）
+       时测的目标点，MTC 却在臂伸出（pitch=11.7°）时执行 → 指令点
+       base(0.432,-0.125,0.895) 实际落到世界 (2.577,1.804,0.794)，罐头在
+       (2.575,2.000,0.780) → 末端前冲 0.196 m，正好是抓取撞飞物体的偏差。
+       几何与底面高度照抄后万向轮（x=-0.177 那两个），保证同一接地平面。 -->
+  <joint name="${prefix}caster_front_joint" type="fixed">
+    <parent link="${prefix}base_link"/>
+    <child link="${prefix}caster_front_link"/>
+    <origin xyz="0.18 0.0 -0.004" rpy="-1.57 0 0"/>
+  </joint>
+  <link name="${prefix}caster_front_link">
+    <collision>
+      <origin xyz="0 0.001 0" rpy="0 0 0"/>
+      <geometry>
+        <box size="0.030 0.009 0.020"/>
+      </geometry>
+    </collision>
+    <inertial>
+      <origin xyz="0 0 0" />
+      <mass value="0.005" />
+      <inertia ixx="0.001" ixy="0.0" ixz="0.0"
+               iyy="0.001" iyz="0.0"
+               izz="0.001" />
+    </inertial>
+  </link>
   <joint name="${prefix}imu_joint" type="fixed">
     <parent link="${prefix}base_link"/>
